File: filer_for_pc.kicad_sch (KiCad schematic)
At the start: 58 parts

Commit message: Update
Other:
- note added: "8"
- note removed: "7"
Changed lines of the file:
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@@
     (stroke (width 0) (type default))
   )
-  (text_box "R9 = 10 Om, R11 = 15kOm, C7 = 300 or 500 pF, L1 = sound speaker, you must solder details directly to speaker. R1, R3, R5, R7, R21, R23, R16, R18 = 33 kOm, R2, R6, R17, R22 = 15 kOm, C2, C5, C15, C18 = 220 pF, C1, C3, C4, C6, C14, C16, C19, C17 = 100 pF.\nR19, R24, R33, R32, R26, R25 = 10MOm, R20, R29, R30, R31, R28, R27 = ~7-8 Om C23, C24 = 33-56 pF,  C12, C13 = 1 mkF. C20, C22, C11, C9 = 100 pF. C18, C15, C21, C10 = 220 pF.\nR12, R14, R4, R15 = 33 kOm, R8, R13 = 15 kOm, Or if you use 224 k instead 1mkF you get cool field(eddy currents also called Foucault's ) shield on ground with about 224v current and 0.04 A.\n\nAll capasitors must be closed by resistors"
+  (text_box "R9 = 10 Om, R11 = 15kOm, C7 = 300 or 500 pF, L1 = sound speaker, you must solder details directly to speaker. R1, R3, R5, R7, R21, R23, R16, R18 = 33 kOm, R2, R6, R17, R22 = 15 kOm, C2, C5, C15, C18 = 220 nF, C1, C3, C4, C6, C14, C16, C19, C17 = 100 nF.\nR19, R24, R33, R32, R26, R25 = 10MOm, R20, R29, R30, R31, R28, R27 = ~7-8 Om C23, C24 = 33-56 pF,  C12, C13 = 100 nF. C20, C22, C11, C9 = 100 nF. C18, C15, C21, C10 = 220 nF.\nR12, R14, R4, R15 = 33 kOm, R8, R13 = 15 kOm. Eddy currents on ground.\n\nAll capasitors must be closed by resistors"
     (at 100.33 127 0) (size 74.93 68.58)
     (stroke (width 0) (type default))
@@
     (effects (font (size 1.27 1.27)) (justify left bottom))
   )
-  (text "7" (at 271.78 194.31 0)
+  (text "8" (at 271.78 194.31 0)
     (effects (font (size 1.27 1.27)) (justify left bottom))
   )

Commit message: Update
Parts:
- removed C8: C,IEC, symbol PCM_Generic:C,IEC
- removed R10: R,IEC, symbol PCM_Generic:R,IEC
Other:
- note added: "10"
- note added: "2023.03.10"
- note added: "modified at 2023.07.11 fix errors in values"
- note removed: "2023.07.03"
- note removed: "8"
- note removed: "C8 = 56 pF R = 10 MOm"
- note removed: "Optional, Experimentral"
Changed lines of the file:
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@@
-    (stroke (width 0) (type default))
-  )
-  (wire (pts (xy 64.77 45.72) (xy 64.77 46.99))
     (stroke (width 0) (type default))
   )
@@
     (stroke (width 0) (type default))
   )
-  (wire (pts (xy 53.34 57.15) (xy 64.77 57.15))
-    (stroke (width 0) (type default))
-  )
   (wire (pts (xy 43.18 99.06) (xy 54.61 99.06))
     (stroke (width 0) (type default))
@@
     (stroke (width 0) (type default))
   )
-  (wire (pts (xy 50.8 35.56) (xy 64.77 35.56))
-    (stroke (width 0) (type default))
-  )
-  (text_box "R9 = 10 Om, R11 = 15kOm, C7 = 300 or 500 pF, L1 = sound speaker, you must solder details directly to speaker. R1, R3, R5, R7, R21, R23, R16, R18 = 33 kOm, R2, R6, R17, R22 = 15 kOm, C2, C5, C15, C18 = 220 nF, C1, C3, C4, C6, C14, C16, C19, C17 = 100 nF.\nR19, R24, R33, R32, R26, R25 = 10MOm, R20, R29, R30, R31, R28, R27 = ~7-8 Om C23, C24 = 33-56 pF,  C12, C13 = 100 nF. C20, C22, C11, C9 = 100 nF. C18, C15, C21, C10 = 220 nF.\nR12, R14, R4, R15 = 33 kOm, R8, R13 = 15 kOm. Eddy currents on ground.\n\nAll capasitors must be closed by resistors"
+  (text_box "R9 = 10 Om, R11 = 1-10MOm, C7 = 600-700 nF, L1 = sound speaker, you must solder details directly to speaker. And I use this about a 3 month. R1, R3, R5, R7, R21, R23, R16, R18 = 33 kOm, R2, R6, R17, R22 = 15 kOm, C2, C5, C15, C18 = 220 nF, C1, C3, C4, C6, C14, C16, C19, C17 = 100 nF.\nR19, R24, R33, R32, R26, R25 = 10MOm, R20, R29, R30, R31, R28, R27 = ~7-8 Om C23, C24 = 33-56 pF,  C12, C13 = 100 nF. C20, C22, C11, C9 = 100 nF. C18, C15, C21, C10 = 220 nF.\nR12, R14, R4, R15 = 33 kOm, R8, R13 = 15 kOm. Eddy currents on ground.\n\nAll capasitors must be closed by resistors"
     (at 100.33 127 0) (size 74.93 68.58)
     (stroke (width 0) (type default))
@@
     (effects (font (size 1.8 1.8)) (justify left top))
   )
-  (text "2023.07.03\n" (at 208.28 194.31 0)
-    (effects (font (size 1.27 1.27)) (justify left bottom))
-  )
-  (text "Optional, Experimentral\n" (at 44.45 31.75 0)
+  (text "2023.03.10\n" (at 208.28 194.31 0)
     (effects (font (size 1.27 1.27)) (justify left bottom))
   )
@@
     (effects (font (size 1.27 1.27)) (justify left bottom))
   )
-  (text "8" (at 271.78 194.31 0)
+  (text "10" (at 271.78 194.31 0)
     (effects (font (size 1.27 1.27)) (justify left bottom))
   )
@@
     (effects (font (size 1.27 1.27)) (justify left bottom))
   )
-  (text "C8 = 56 pF R = 10 MOm\n" (at 35.56 48.26 0)
+  (text "modified at 2023.07.11 fix errors in values" (at 217.17 172.72 0)
     (effects (font (size 1.27 1.27)) (justify left bottom))
   )
   (label "Ground must use shieded cable" (at 162.56 106.68 0) (fields_autoplaced)
     (effects (font (size 1.4 1.4)) (justify left bottom))
-  )
-  (global_label "Line" (shape input) (at 50.8 35.56 180) (fields_autoplaced)
-    (effects (font (size 1.27 1.27)) (justify right))
-    (property "Intersheetrefs" "${INTERSHEET_REFS}" (at 44.0237 35.56 0)
-      (effects (font (size 1.27 1.27)) (justify right) hide)
-    )
-  )
-  (global_label "Neutral" (shape input) (at 53.34 57.15 180) (fields_autoplaced)
-    (effects (font (size 1.27 1.27)) (justify right))
-    (property "Intersheetrefs" "${INTERSHEET_REFS}" (at 43.54 57.15 0)
-      (effects (font (size 1.27 1.27)) (justify right) hide)
-    )
   )
   (global_label "220 AC" (shape input) (at 99.06 31.75 180) (fields_autoplaced)
@@
     )
   )
-  (symbol (lib_id "PCM_Generic:C,IEC") (at 64.77 40.64 0) (unit 1)
-    (in_bom yes) (on_board yes) (dnp no) (fields_autoplaced)
-    (property "Reference" "C8" (at 60.96 38.1 0)
-      (effects (font (size 2.54 2.54)) (justify right))
-    )
-    (property "Value" "C,IEC" (at 60.96 41.91 0)
-      (effects (font (size 2.54 2.54)) (justify right))
-    )
-    (property "Footprint" "" (at 64.77 40.64 0)
-      (effects (font (size 2.54 2.54)) hide)
-    )
-    (property "Datasheet" "" (at 64.77 40.64 0)
-      (effects (font (size 2.54 2.54)) hide)
-    )
-    (property "Indicator" "" (at 60.96 45.085 0)
-      (effects (font (size 1.27 1.27)) (justify right))
-    )
-    (property "Field5" "" (at 64.77 40.64 0)
-      (effects (font (size 1.27 1.27)) hide)
-    )
-    (pin "1")
-    (pin "2")
-    (instances
-      (project "filer_for_pc"
-        (path "/cdde10a9-1f5d-4493-ba10-a349138f6d4d"
-          (reference "C8") (unit 1)
-        )
-      )
-    )
-  )
   (symbol (lib_id "PCM_Generic-50:C,IEC") (at 229.87 62.23 270) (unit 1)
     (in_bom yes) (on_board yes) (dnp no) (fields_autoplaced)
@@
         )
       )
-    )
-  )
-  (symbol (lib_id "PCM_Generic:R,IEC") (at 64.77 52.07 0) (unit 1)
-    (in_bom yes) (on_board yes) (dnp no) (fields_autoplaced)
-    (property "Reference" "R10" (at 67.31 50.8 0)
-      (effects (font (size 2.54 2.54)) (justify left))
-    )
-    (property "Value" "R,IEC" (at 67.31 54.61 0)
-      (effects (font (size 2.54 2.54)) (justify left))
-    )
-    (property "Footprint" "" (at 64.77 52.07 0)
-      (effects (font (size 2.54 2.54)) hide)
-    )
-    (property "Datasheet" "" (at 64.77 52.07 0)
-      (effects (font (size 2.54 2.54)) hide)
-    )
-    (property "Indicator" "+" (at 62.23 49.53 0)
-      (effects (font (size 1.27 1.27)) hide)
-    )
-    (pin "1")
-    (pin "2")
-    (instances
-      (project "filer_for_pc"
-        (path "/cdde10a9-1f5d-4493-ba10-a349138f6d4d"
-          (reference "R10") (unit 1)
-        )
-      )

Commit message: Upgrade
Parts:
- removed C1, C6: C,IEC, symbol PCM_Generic:C,IEC
- removed C2, C3, C7, C8: C,IEC, symbol PCM_Generic-50:C,IEC
- removed R1 (x3), R2, R3, R4, R5, R6: R,IEC, symbol PCM_Generic:R,IEC
- added R10: R,IEC, symbol PCM_Generic:R,IEC
Connections:
- net at R1.2 (-), R1.2 (-), R1.2 (-)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: now also R10.1 (+)
- net at C2.1 (+), R1.2 (-), R2.1 (+): no longer R25.2 (-)
- net at R25.1 (+): now also R26.2 (-)
- net at C1.2 (-), C1.2 (-), R1.1 (+)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: now also R10.2 (-)
Other:
- note added: "11"
- note removed: "10"
- moved on the sheet: R25, R26

Commit message: Upgrade
Parts:
- removed R1 (x3): R,IEC, symbol PCM_Generic:R,IEC
- added R32: R,IEC, symbol PCM_Generic:R,IEC
- renumbered R10 to R19
Connections:
- net Ground: no longer R1.1 (+), R1.2 (-), R1.2 (-)
- net at C2.1 (+), R2.1 (+): no longer R1.2 (-)
- net at C1.2 (-), C1.2 (-), R1.1 (+)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: now also R1.2 (-)
- net at C1.1 (+), C2.1 (+), R2.1 (+): now also R32.1 (+)
- net at R25.1 (+): now also R32.2 (-); no longer R26.2 (-)
- net at R25.2 (-): now also R26.2 (-)
- net at C1.2 (-), C3.2 (-), R3.2 (-): now also R26.1 (+)
- new net: R1.1 (+), R1.2 (-), R1.2 (-)
Other:
- moved on the sheet: R1, R25

Commit message: Upgrade
Parts:
- added C1 (x2): C,IEC, symbol PCM_Generic:C,IEC
- added R1: R,IEC, symbol PCM_Generic:R,IEC
Connections:
- new net: C1.1 (+), C1.2 (-), R1.2 (-)
Other:
- note added: "modified at 2023.07.21"
- note removed: "modified at 2023.07.11 fix errors in values"
- moved on the sheet: R25, R26

Commit message: Upgrade
Parts:
- added R2, R3: R,IEC, symbol PCM_Generic:R,IEC
Connections:
- net at R1.1 (+): now also R2.1 (+), R3.1 (+)
- net at C1.1 (+), C1.2 (-), R1.2 (-): now also R2.2 (-), R3.2 (-)
Other:
- note added: "modified at 2023.07.22"
- note removed: "modified at 2023.07.21"
Changed lines of the file:
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@@
   (junction (at 76.2 120.65) (diameter 0) (color 0 0 0 0)
   )
+  (junction (at 111.76 59.69) (diameter 0) (color 0 0 0 0)
+  )
   (junction (at 54.61 87.63) (diameter 0) (color 0 0 0 0)
   )
@@
   (junction (at 228.6 134.62) (diameter 0) (color 0 0 0 0)
   )
+  (junction (at 137.16 90.17) (diameter 0) (color 0 0 0 0)
+  )
   (junction (at 223.52 95.25) (diameter 0) (color 0 0 0 0)
   )
@@
   (junction (at 269.24 62.23) (diameter 0) (color 0 0 0 0)
   )
+  (junction (at 137.16 63.5) (diameter 0) (color 0 0 0 0)
+  )
   (junction (at 54.61 152.4) (diameter 0) (color 0 0 0 0)
   )
@@
   (junction (at 34.29 120.65) (diameter 0) (color 0 0 0 0)
   )
-  (wire (pts (xy 137.16 59.69) (xy 137.16 96.52))
+  (wire (pts (xy 137.16 59.69) (xy 137.16 63.5))
     (stroke (width 0) (type default))
   )
@@
     (stroke (width 0) (type default))
   )
+  (wire (pts (xy 111.76 55.88) (xy 128.27 55.88))
+    (stroke (width 0) (type default))
+  )
   (wire (pts (xy 245.11 81.28) (xy 245.11 92.71))
     (stroke (width 0) (type default))
@@
     (stroke (width 0) (type default))
   )
+  (wire (pts (xy 80.01 90.17) (xy 106.68 90.17))
+    (stroke (width 0) (type default))
+  )
   (wire (pts (xy 49.53 132.08) (xy 49.53 120.65))
     (stroke (width 0) (type default))
@@
     (stroke (width 0) (type default))
   )
+  (wire (pts (xy 138.43 55.88) (xy 138.43 63.5))
+    (stroke (width 0) (type default))
+  )
   (wire (pts (xy 54.61 152.4) (xy 54.61 154.94))
     (stroke (width 0) (type default))
@@
     (stroke (width 0) (type default))
   )
-  (wire (pts (xy 106.68 59.69) (xy 116.84 59.69))
+  (wire (pts (xy 106.68 59.69) (xy 111.76 59.69))
     (stroke (width 0) (type default))
   )
@@
     (stroke (width 0) (type default))
   )
+  (wire (pts (xy 138.43 63.5) (xy 137.16 63.5))
+    (stroke (width 0) (type default))
+  )
   (wire (pts (xy 76.2 107.95) (xy 38.1 107.95))
     (stroke (width 0) (type default))
@@
     (stroke (width 0) (type default))
   )
+  (wire (pts (xy 111.76 59.69) (xy 111.76 55.88))
+    (stroke (width 0) (type default))
+  )
   (wire (pts (xy 54.61 139.7) (xy 54.61 142.24))
     (stroke (width 0) (type default))
@@
     (stroke (width 0) (type default))
   )
+  (wire (pts (xy 106.68 59.69) (xy 80.01 59.69))
+    (stroke (width 0) (type default))
+  )
+  (wire (pts (xy 116.84 90.17) (xy 137.16 90.17))
+    (stroke (width 0) (type default))
+  )
   (wire (pts (xy 100.33 120.65) (xy 135.89 120.65))
     (stroke (width 0) (type default))
@@
     (stroke (width 0) (type default))
   )
+  (wire (pts (xy 80.01 59.69) (xy 80.01 90.17))
+    (stroke (width 0) (type default))
+  )
+  (wire (pts (xy 137.16 63.5) (xy 137.16 90.17))
+    (stroke (width 0) (type default))
+  )
   (wire (pts (xy 233.68 54.61) (xy 247.65 54.61))
     (stroke (width 0) (type default))
@@
     (stroke (width 0) (type default))
   )
+  (wire (pts (xy 137.16 90.17) (xy 137.16 96.52))
+    (stroke (width 0) (type default))
+  )
   (wire (pts (xy 72.39 153.67) (xy 76.2 153.67))
     (stroke (width 0) (type default))
@@
     (stroke (width 0) (type default))
   )
+  (wire (pts (xy 111.76 59.69) (xy 116.84 59.69))
+    (stroke (width 0) (type default))
+  )
   (wire (pts (xy 72.39 104.14) (xy 101.6 104.14))
     (stroke (width 0) (type default))
@@
     (stroke (width 0) (type default))
   )
-  (text_box "R9 = 10 Om, R11 = 1-10MOm, C7 = 600-700 nF, L1 = sound speaker, you must solder details directly to speaker. And I use this about a 3 month. R1, R3, R5, R7, R21, R23, R16, R18 = 33 kOm, R2, R6, R17, R22 = 15 kOm, C2, C5, C15, C18 = 220 nF, C1, C3, C4, C6, C14, C16, C19, C17 = 100 nF.\nR19, R24, R33, R32, R26, R25 = 10MOm, R1, R20, R29, R30, R31, R28, R27 = ~7-8-10 Om C23, C24 = 10-1000 nF,  C12, C13 = 100 nF. C20, C22, C11, C9 = 100 nF. C18, C15, C21, C10 = 220 nF.\nR12, R14, R4, R15 = 33 kOm, R8, R13 = 15 kOm. Eddy currents on ground. C1, C2 = 16 pF.\n\nAll capasitors must be closed by resistors"
+  (text_box "R9 = 10 Om, R11 = 1-10MOm, C7 = 600-700 nF, L1 = sound speaker, you must solder details directly to speaker. And I use this about a 3 month.\nC15, C18 = 220 nF, C14, C16, C19, C17 = 100 nF. R2, R19, R24, R33, R32, R26, R25 = 10MOm, \nR1, R20, R29, R30, R31, R28, R27 = ~7-8-10 Om C23, C24 = 10-1000 nF, R3 = 70Om 1GHz - or 50 Om 2GHz\nC12, C13 = 100 nF. C20, C22, C11, C9 = 100 nF. C18, C15, C21, C10 = 220 nF.\nR12, R14, R4, R15 = 33 kOm, R8, R13 = 15 kOm. Eddy currents on ground. C1, C2 = 16 pF.\n\nAll capasitors must be closed by resistors\n"
     (at 100.33 127 0) (size 74.93 68.58)
     (stroke (width 0) (type default))
@@
     (effects (font (size 1.27 1.27)) (justify left bottom))
   )
-  (text "modified at 2023.07.21\n" (at 217.17 172.72 0)
+  (text "modified at 2023.07.22\n\n" (at 217.17 172.72 0)
     (effects (font (size 1.27 1.27)) (justify left bottom))
   )
@@
     )
   )
+  (symbol (lib_id "PCM_Generic:R,IEC") (at 111.76 90.17 270) (unit 1)
+    (in_bom yes) (on_board yes) (dnp no) (fields_autoplaced)
+    (property "Reference" "R3" (at 111.76 80.01 90)
+      (effects (font (size 2.54 2.54)))
+    )
+    (property "Value" "R,IEC" (at 111.76 85.09 90)
+      (effects (font (size 2.54 2.54)))
+    )
+    (property "Footprint" "" (at 111.76 90.17 0)
+      (effects (font (size 2.54 2.54)) hide)
+    )
+    (property "Datasheet" "" (at 111.76 90.17 0)
+      (effects (font (size 2.54 2.54)) hide)
+    )
+    (property "Indicator" "+" (at 114.3 87.63 0)
+      (effects (font (size 1.27 1.27)) hide)
+    )
+    (pin "1")
+    (pin "2")
+    (instances
+      (project "filer_for_pc"
+        (path "/cdde10a9-1f5d-4493-ba10-a349138f6d4d"
+          (reference "R3") (unit 1)
+        )
+      )
+    )
+  )
   (symbol (lib_id "PCM_Generic-50:C,IEC") (at 229.87 62.23 270) (unit 1)
     (in_bom yes) (on_board yes) (dnp no) (fields_autoplaced)
@@
         )
       )
+    )
+  )
+  (symbol (lib_id "PCM_Generic:R,IEC") (at 133.35 55.88 270) (unit 1)
+    (in_bom yes) (on_board yes) (dnp no) (fields_autoplaced)
+    (property "Reference" "R2" (at 133.35 45.72 90)
+      (effects (font (size 2.54 2.54)))
+    )
+    (property "Value" "R,IEC" (at 133.35 50.8 90)
+      (effects (font (size 2.54 2.54)))
+    )
+    (property "Footprint" "" (at 133.35 55.88 0)
+      (effects (font (size 2.54 2.54)) hide)
+    )
+    (property "Datasheet" "" (at 133.35 55.88 0)
+      (effects (font (size 2.54 2.54)) hide)
+    )
+    (property "Indicator" "+" (at 135.89 53.34 0)
+      (effects (font (size 1.27 1.27)) hide)
+    )
+    (pin "1")
+    (pin "2")
+    (instances
+      (project "filer_for_pc"
+        (path "/cdde10a9-1f5d-4493-ba10-a349138f6d4d"
+          (reference "R2") (unit 1)
+        )
+      )
