File: filer_for_pc.kicad_sch (KiCad schematic)
At the start: 46 parts

Commit message: Upgrade
Parts:
- removed R2, R32: R,IEC, symbol PCM_Generic:R,IEC
Connections:
- net at R25.2 (-): no longer R26.2 (-)
- net at C1.2 (-), C3.2 (-), R3.2 (-): no longer R26.1 (+)
Other:
- moved on the sheet: R26
Changed lines of the file:
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@@
   (junction (at 219.71 134.62) (diameter 0) (color 0 0 0 0)
   )
-  (junction (at 247.65 66.04) (diameter 0) (color 0 0 0 0)
-  )
   (junction (at 72.39 153.67) (diameter 0) (color 0 0 0 0)
   )
@@
   (junction (at 223.52 81.28) (diameter 0) (color 0 0 0 0)
   )
-  (junction (at 154.94 45.72) (diameter 0) (color 0 0 0 0)
-  )
   (junction (at 54.61 99.06) (diameter 0) (color 0 0 0 0)
   )
   (junction (at 76.2 120.65) (diameter 0) (color 0 0 0 0)
   )
-  (junction (at 111.76 59.69) (diameter 0) (color 0 0 0 0)
-  )
   (junction (at 54.61 87.63) (diameter 0) (color 0 0 0 0)
   )
@@
   (junction (at 223.52 106.68) (diameter 0) (color 0 0 0 0)
   )
-  (junction (at 154.94 83.82) (diameter 0) (color 0 0 0 0)
-  )
   (junction (at 228.6 134.62) (diameter 0) (color 0 0 0 0)
   )
@@
   (junction (at 100.33 120.65) (diameter 0) (color 0 0 0 0)
   )
-  (junction (at 247.65 35.56) (diameter 0) (color 0 0 0 0)
-  )
   (junction (at 269.24 62.23) (diameter 0) (color 0 0 0 0)
   )
-  (junction (at 137.16 63.5) (diameter 0) (color 0 0 0 0)
-  )
   (junction (at 54.61 152.4) (diameter 0) (color 0 0 0 0)
   )
@@
   (junction (at 34.29 120.65) (diameter 0) (color 0 0 0 0)
   )
-  (wire (pts (xy 137.16 59.69) (xy 137.16 63.5))
+  (wire (pts (xy 137.16 59.69) (xy 137.16 90.17))
     (stroke (width 0) (type default))
   )
@@
     (stroke (width 0) (type default))
   )
-  (wire (pts (xy 111.76 55.88) (xy 128.27 55.88))
-    (stroke (width 0) (type default))
-  )
   (wire (pts (xy 245.11 81.28) (xy 245.11 92.71))
     (stroke (width 0) (type default))
   )
-  (wire (pts (xy 154.94 45.72) (xy 175.26 45.72))
-    (stroke (width 0) (type default))
-  )
   (wire (pts (xy 242.57 153.67) (xy 228.6 153.67))
     (stroke (width 0) (type default))
@@
     (stroke (width 0) (type default))
   )
-  (wire (pts (xy 247.65 25.4) (xy 247.65 35.56))
-    (stroke (width 0) (type default))
-  )
   (wire (pts (xy 266.7 76.2) (xy 269.24 76.2))
     (stroke (width 0) (type default))
@@
     (stroke (width 0) (type default))
   )
-  (wire (pts (xy 154.94 45.72) (xy 154.94 57.15))
-    (stroke (width 0) (type default))
-  )
   (wire (pts (xy 106.68 40.64) (xy 106.68 48.26))
     (stroke (width 0) (type default))
@@
     (stroke (width 0) (type default))
   )
-  (wire (pts (xy 173.99 73.66) (xy 173.99 66.04))
-    (stroke (width 0) (type default))
-  )
   (wire (pts (xy 48.26 139.7) (xy 54.61 139.7))
     (stroke (width 0) (type default))
@@
     (stroke (width 0) (type default))
   )
-  (wire (pts (xy 154.94 67.31) (xy 154.94 83.82))
+  (wire (pts (xy 154.94 67.31) (xy 154.94 92.71))
     (stroke (width 0) (type default))
   )
@@
     (stroke (width 0) (type default))
   )
-  (wire (pts (xy 154.94 31.75) (xy 154.94 45.72))
+  (wire (pts (xy 154.94 31.75) (xy 154.94 57.15))
     (stroke (width 0) (type default))
   )
@@
     (stroke (width 0) (type default))
   )
-  (wire (pts (xy 138.43 55.88) (xy 138.43 63.5))
-    (stroke (width 0) (type default))
-  )
   (wire (pts (xy 54.61 152.4) (xy 54.61 154.94))
     (stroke (width 0) (type default))
@@
     (stroke (width 0) (type default))
   )
-  (wire (pts (xy 106.68 59.69) (xy 111.76 59.69))
-    (stroke (width 0) (type default))
-  )
   (wire (pts (xy 38.1 135.89) (xy 76.2 135.89))
     (stroke (width 0) (type default))
   )
-  (wire (pts (xy 138.43 63.5) (xy 137.16 63.5))
-    (stroke (width 0) (type default))
-  )
   (wire (pts (xy 76.2 107.95) (xy 38.1 107.95))
     (stroke (width 0) (type default))
@@
     (stroke (width 0) (type default))
   )
-  (wire (pts (xy 154.94 83.82) (xy 173.99 83.82))
-    (stroke (width 0) (type default))
-  )
   (wire (pts (xy 269.24 62.23) (xy 269.24 76.2))
     (stroke (width 0) (type default))
@@
     (stroke (width 0) (type default))
   )
-  (wire (pts (xy 111.76 59.69) (xy 111.76 55.88))
-    (stroke (width 0) (type default))
-  )
   (wire (pts (xy 54.61 139.7) (xy 54.61 142.24))
     (stroke (width 0) (type default))
@@
     (stroke (width 0) (type default))
   )
-  (wire (pts (xy 175.26 35.56) (xy 184.15 35.56))
-    (stroke (width 0) (type default))
-  )
   (wire (pts (xy 43.18 165.1) (xy 54.61 165.1))
     (stroke (width 0) (type default))
@@
     (stroke (width 0) (type default))
   )
-  (wire (pts (xy 137.16 63.5) (xy 137.16 90.17))
-    (stroke (width 0) (type default))
-  )
   (wire (pts (xy 233.68 54.61) (xy 247.65 54.61))
     (stroke (width 0) (type default))
   )
-  (wire (pts (xy 184.15 25.4) (xy 247.65 25.4))
-    (stroke (width 0) (type default))
-  )
   (wire (pts (xy 228.6 148.59) (xy 228.6 153.67))
     (stroke (width 0) (type default))
@@
     (stroke (width 0) (type default))
   )
-  (wire (pts (xy 173.99 66.04) (xy 247.65 66.04))
-    (stroke (width 0) (type default))
-  )
   (wire (pts (xy 137.16 96.52) (xy 160.02 96.52))
     (stroke (width 0) (type default))
@@
     (stroke (width 0) (type default))
   )
-  (wire (pts (xy 111.76 59.69) (xy 116.84 59.69))
+  (wire (pts (xy 106.68 59.69) (xy 116.84 59.69))
     (stroke (width 0) (type default))
   )
@@
     (stroke (width 0) (type default))
   )
-  (wire (pts (xy 184.15 35.56) (xy 184.15 25.4))
-    (stroke (width 0) (type default))
-  )
   (wire (pts (xy 76.2 120.65) (xy 90.17 120.65))
     (stroke (width 0) (type default))
@@
   )
   (wire (pts (xy 72.39 139.7) (xy 72.39 153.67))
-    (stroke (width 0) (type default))
-  )
-  (wire (pts (xy 154.94 83.82) (xy 154.94 92.71))
     (stroke (width 0) (type default))
   )
@@
     (effects (font (size 1.4 1.4)) (justify left bottom))
   )
-  (label "2023{slash}07{slash}17" (at 227.33 185.42 0) (fields_autoplaced)
+  (label "2023{slash}08{slash}09" (at 227.33 185.42 0) (fields_autoplaced)
     (effects (font (size 1.27 1.27)) (justify left bottom))
   )
@@
     )
   )
-  (symbol (lib_id "PCM_Generic:R,IEC") (at 173.99 78.74 0) (unit 1)
-    (in_bom yes) (on_board yes) (dnp no) (fields_autoplaced)
-    (property "Reference" "R26" (at 176.53 76.1999 0)
+  (symbol (lib_id "PCM_Generic:R,IEC") (at 118.11 102.87 0) (unit 1)
+    (in_bom yes) (on_board yes) (dnp no) (fields_autoplaced)
+    (property "Reference" "R26" (at 120.65 100.3299 0)
       (effects (font (size 2.54 2.54)) (justify left))
     )
-    (property "Value" "R,IEC" (at 176.53 81.2799 0)
+    (property "Value" "R,IEC" (at 120.65 105.4099 0)
       (effects (font (size 2.54 2.54)) (justify left))
     )
-    (property "Footprint" "" (at 173.99 78.74 0)
-      (effects (font (size 2.54 2.54)) hide)
-    )
-    (property "Datasheet" "" (at 173.99 78.74 0)
-      (effects (font (size 2.54 2.54)) hide)
-    )
-    (property "Indicator" "+" (at 171.45 76.2 0)
+    (property "Footprint" "" (at 118.11 102.87 0)
+      (effects (font (size 2.54 2.54)) hide)
+    )
+    (property "Datasheet" "" (at 118.11 102.87 0)
+      (effects (font (size 2.54 2.54)) hide)
+    )
+    (property "Indicator" "+" (at 115.57 100.33 0)
       (effects (font (size 1.27 1.27)) hide)
     )
@@
     )
   )
-  (symbol (lib_id "PCM_Generic:R,IEC") (at 175.26 40.64 0) (unit 1)
-    (in_bom yes) (on_board yes) (dnp no) (fields_autoplaced)
-    (property "Reference" "R32" (at 177.8 38.0999 0)
-      (effects (font (size 2.54 2.54)) (justify left))
-    )
-    (property "Value" "R,IEC" (at 177.8 43.1799 0)
-      (effects (font (size 2.54 2.54)) (justify left))
-    )
-    (property "Footprint" "" (at 175.26 40.64 0)
-      (effects (font (size 2.54 2.54)) hide)
-    )
-    (property "Datasheet" "" (at 175.26 40.64 0)
-      (effects (font (size 2.54 2.54)) hide)
-    )
-    (property "Indicator" "+" (at 172.72 38.1 0)
-      (effects (font (size 1.27 1.27)) hide)
-    )
-    (pin "1")
-    (pin "2")
-    (instances
-      (project "filer_for_pc"
-        (path "/cdde10a9-1f5d-4493-ba10-a349138f6d4d"
-          (reference "R32") (unit 1)
-        )
-      )
-    )
-  )
   (symbol (lib_id "PCM_Generic:R,IEC") (at 228.6 143.51 0) (unit 1)
     (in_bom yes) (on_board yes) (dnp no) (fields_autoplaced)
@@
         )
       )
-    )
-  )
-  (symbol (lib_id "PCM_Generic:R,IEC") (at 133.35 55.88 270) (unit 1)
-    (in_bom yes) (on_board yes) (dnp no) (fields_autoplaced)
-    (property "Reference" "R2" (at 133.35 45.72 90)
-      (effects (font (size 2.54 2.54)))
-    )
-    (property "Value" "R,IEC" (at 133.35 50.8 90)
-      (effects (font (size 2.54 2.54)))
-    )
-    (property "Footprint" "" (at 133.35 55.88 0)
-      (effects (font (size 2.54 2.54)) hide)
-    )
-    (property "Datasheet" "" (at 133.35 55.88 0)
-      (effects (font (size 2.54 2.54)) hide)
-    )
-    (property "Indicator" "+" (at 135.89 53.34 0)
-      (effects (font (size 1.27 1.27)) hide)
-    )
-    (pin "1")
-    (pin "2")
-    (instances
-      (project "filer_for_pc"
-        (path "/cdde10a9-1f5d-4493-ba10-a349138f6d4d"
-          (reference "R2") (unit 1)
-        )
-      )

Commit message: Added updates
Parts:
- added C3: C,IEC, symbol PCM_Generic:C,IEC
- added L2: L,current,IEC, symbol PCM_Generic:L,current,IEC
- added R2, R5, R6, R7: R,IEC, symbol PCM_Generic:R,IEC
Connections:
- net at R9.2 (-): now also R6.2 (-)
- new net: C3.1 (+), L2.1 (+), R2.1 (+), R5.1 (+)
- new net: C3.2 (-), L2.2 (-), R5.2 (-)
- new net: R2.2 (-), R6.1 (+)
Other:
- moved on the sheet: C1, C2, C3, C7, L1, R1, R11, R2, R25, R3, R9
